File: hw/lpf1/lpf.kicad_sch (KiCad schematic)
At the start: 39 parts, among them Q1 MMBT3904, Q2 MMBT3904

Commit message: Sending QRP PA/LPF boards to JLC
Other:
- company: (none) -> Bruce MacKinnon, KC1FSZ
- title: (none) -> Low Pass Filter Board 1
Changed lines of the file:
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@@
 	(generator "eeschema")
 	(generator_version "8.0")
-	(paper "A4")
+	(paper "USLetter")
+	(title_block
+		(title "Low Pass Filter Board 1")
+		(date "2025-02-21")
+		(rev "1")
+		(company "Bruce MacKinnon, KC1FSZ")
+		(comment 1 "Copyright (C) Bruce MacKinnon, 2025")
+		(comment 2 "NOT FOR COMMERCIAL USE")
+	)
 	(junction
 		(at 132.08 116.84)
