File: hw/lpf1/lpf1.kicad_pcb (KiCad board)
At the start: 2 copper layers, 100 x 35 mm, 51 parts, among them J1 Conn_Coaxial, J2 Conn_Coaxial, J3 Conn_Coaxial, J4 Conn_01x05, K1 G6E, Q1 MMBT3904, Q2 MMBT3904, Q3 MMBT3904

Commit message: Layout complete
Parts:
- added C17: 0.1u, Capacitor_SMD:C_0805_2012Metric_Pad1.18x1.45mm_HandSolder, F.Cu at (208.5, 74.5)
- added C18: 0.1u, Capacitor_SMD:C_0805_2012Metric_Pad1.18x1.45mm_HandSolder, F.Cu at (203.0, 74.5)
- added D6: BAT46W, Diode_SMD:D_SOD-123, F.Cu at (208.5, 72.0)
- added D7: BAT46W, Diode_SMD:D_SOD-123, F.Cu at (203.0, 72.0)
- added J5: Conn_01x04, Connector_PinHeader_2.54mm:PinHeader_1x04_P2.54mm_Vertical, F.Cu at (209.5, 81.5)
- added R5: 47, Resistor_SMD:R_0805_2012Metric_Pad1.20x1.40mm_HandSolder, F.Cu at (208.5, 69.5)
- added R6: 47, Resistor_SMD:R_0805_2012Metric_Pad1.20x1.40mm_HandSolder, F.Cu at (203.0, 69.5)
- added R7: 220k, Resistor_SMD:R_0805_2012Metric_Pad1.20x1.40mm_HandSolder, F.Cu at (208.5, 77.0)
- added R8: 220k, Resistor_SMD:R_0805_2012Metric_Pad1.20x1.40mm_HandSolder, F.Cu at (203.0, 77.0)
- added T1: ~, bruce-footprints:Dual Transformer 1, F.Cu at (205.0, 55.0)
- C10: value 0.1uF -> 390
- C11: value 180p -> 270p
- C12: value 390p -> 180p
- C13: value 390 -> 0.1uF
- C14: value 180p -> 0.1uF
- C6: value 270p -> 180p
- C8: value 680p -> 390p
- C9: value 0.1uF -> 680p
- L1, L3: value 1.38uH -> 47uH; footprint bruce-footprints:FT37-43 Unifilar -> Inductor_SMD:L_0805_2012Metric_Pad1.15x1.40mm_HandSolder
- L11: value 0.904u -> 47uH; footprint bruce-footprints:FT37-43 Unifilar -> Inductor_SMD:L_0805_2012Metric_Pad1.15x1.40mm_HandSolder
- L12: value 0.773u -> 47uH; footprint bruce-footprints:FT37-43 Unifilar -> Inductor_SMD:L_0805_2012Metric_Pad1.15x1.40mm_HandSolder
- L2: value 1.7uH -> 47uH; footprint bruce-footprints:FT37-43 Unifilar -> Inductor_SMD:L_0805_2012Metric_Pad1.15x1.40mm_HandSolder
- L5, L9: value 47uH -> 1.38uH; footprint Inductor_SMD:L_0805_2012Metric_Pad1.15x1.40mm_HandSolder -> bruce-footprints:FT37-43 Unifilar
- L6: value 47uH -> 0.773u; footprint Inductor_SMD:L_0805_2012Metric_Pad1.15x1.40mm_HandSolder -> bruce-footprints:FT37-43 Unifilar
- L7: value 47uH -> 1.7uH; footprint Inductor_SMD:L_0805_2012Metric_Pad1.15x1.40mm_HandSolder -> bruce-footprints:FT37-43 Unifilar
- L8: value 47uH -> 0.904u; footprint Inductor_SMD:L_0805_2012Metric_Pad1.15x1.40mm_HandSolder -> bruce-footprints:FT37-43 Unifilar
- moved Q1 43.5 mm to (150.6, 60.1)
- moved Q2 43.4 mm to (150.6, 75.1)
- moved R2 43.4 mm to (150.6, 56.1), turned to 0 degrees
- moved R3 43.3 mm to (150.6, 71.5)
- moved D3 42.3 mm to (192.5, 59.5), turned to 180 degrees
- moved C11 36.2 mm to (191.5, 67.0)
- moved L9 36.0 mm to (183.9, 60.5), turned to 90 degrees
- moved H4 35.0 mm to (218.0, 82.0)
- moved L4 34.2 mm to (159.0, 77.5), turned to 180 degrees
- moved C1 29.4 mm to (159.0, 70.5), turned to 180 degrees
- moved C9 28.8 mm to (181.9, 67.0), turned to 0 degrees
- moved C10 28.3 mm to (181.9, 82.5), turned to 0 degrees
- moved C2 28.2 mm to (159.0, 55.0), turned to 180 degrees
- moved D1 27.6 mm to (159.0, 59.5), turned to 0 degrees
- moved L11 25.9 mm to (192.0, 62.0), turned to 0 degrees
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Connections:
- C1 pad 1: Net-(D1-A) -> Net-(D2-A)
- C1 pad 2: LPF_OUT -> LPF_IN
- C10 pad 2: Net-(D3-K) -> GND
- C11 pad 1: Net-(C10-Pad1) -> Net-(C11-Pad1)
- C13 pad 1: Net-(C13-Pad1) -> Net-(C11-Pad1)
- C13 pad 2: GND -> Net-(D3-K)
- C14 pad 1: Net-(C14-Pad1) -> Net-(C12-Pad1)
- C14 pad 2: GND -> Net-(D4-K)
- C15 pad 1: Net-(C14-Pad1) -> Net-(D4-A)
- C15 pad 2: Net-(D4-K) -> LPF_OUT
- C16 pad 1: Net-(D4-A) -> Net-(D3-A)
- C2 pad 1: Net-(C2-Pad1) -> Net-(D1-A)
- C2 pad 2: Net-(D1-K) -> LPF_IN
- C3 pad 2: Net-(D2-K) -> Net-(D1-K)
- C4 pad 1: Net-(D2-A) -> Net-(C4-Pad1)
- C4 pad 2: /RF_A -> Net-(D2-K)
- C6 pad 1: Net-(C2-Pad1) -> Net-(C4-Pad1)
- C9 pad 1: Net-(D3-A) -> Net-(C9-Pad1)
- C9 pad 2: /RF_A -> GND
- J3 pad 1: LPF_OUT -> ANT
- K1 pad 7: /RF_A -> LPF_IN
- L1 pad 1: Net-(C3-Pad1) -> Net-(D1-A)
- L1 pad 2: Net-(C7-Pad1) -> Net-(L1-Pad2)
- L11 pad 1: Net-(C12-Pad1) -> Net-(Q1-C)
- L11 pad 2: Net-(C13-Pad1) -> Net-(D3-K)
- L12 pad 1: Net-(C13-Pad1) -> Net-(Q2-C)
- L12 pad 2: Net-(C14-Pad1) -> Net-(D4-K)
- L13 pad 1: Net-(Q2-C) -> Net-(D3-A)
- L13 pad 2: Net-(D4-K) -> Net-(L1-Pad2)
- L14 pad 2: Net-(L14-Pad2) -> Net-(L1-Pad2)
- L2 pad 1: Net-(C7-Pad1) -> Net-(D2-A)
- L2 pad 2: Net-(C8-Pad1) -> Net-(L1-Pad2)
- L3 pad 1: Net-(C8-Pad1) -> Net-(Q1-C)
- L3 pad 2: Net-(C2-Pad1) -> Net-(D1-K)
- L4 pad 1: Net-(D1-A) -> Net-(Q2-C)
- L4 pad 2: Net-(L14-Pad2) -> Net-(D2-K)
- L5 pad 1: Net-(Q1-C) -> Net-(C3-Pad1)
- L5 pad 2: Net-(D1-K) -> Net-(C7-Pad1)
- L6 pad 1: Net-(D2-A) -> Net-(C4-Pad1)
- L6 pad 2: Net-(L14-Pad2) -> Net-(C8-Pad1)
- L7 pad 1: Net-(Q1-C) -> Net-(C7-Pad1)
- L7 pad 2: Net-(D2-K) -> Net-(C9-Pad1)
- L8 pad 1: Net-(D3-A) -> Net-(C8-Pad1)
- L8 pad 2: Net-(L14-Pad2) -> Net-(C10-Pad1)
- L9 pad 1: Net-(Q2-C) -> Net-(C9-Pad1)
- L9 pad 2: Net-(D3-K) -> Net-(C11-Pad1)
- R1 pad 2: Net-(L14-Pad2) -> Net-(L1-Pad2)
Routing:
- net Net-(L1-Pad2): track 0.00 -> 91.0 mm, vias 0 -> 5
- net Net-(Q2-C): track 0.00 -> 43.5 mm, vias 0 -> 3
- net Net-(Q1-C): track 0.00 -> 43.4 mm, vias 0 -> 3
- net LPF_IN: track 0.00 -> 40.8 mm
- net /RF_A: track 38.5 -> 0.00 mm
- net GND: track 0.00 -> 27.3 mm, vias 0 -> 17
- net Net-(D7-A): track 0.00 -> 23.5 mm
- net ANT: track 0.00 -> 22.1 mm
- net LPF_SEL1: track 0.00 -> 20.4 mm, vias 0 -> 1
- net Net-(D6-A): track 0.00 -> 18.0 mm, vias 0 -> 1
- net LPF_SEL0: track 0.00 -> 11.3 mm
- net Net-(C14-Pad1): track 11.2 -> 0.00 mm
- net +5V: track 16.4 -> 5.33 mm, vias 0 -> 1
- net Net-(C2-Pad1): track 11.0 -> 0.00 mm
- net V_REV: track 0.00 -> 10.8 mm
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- added copper zone on In2.Cu, net +5V
- added copper zone on In1.Cu, net GND
Other:
- copper layers 2 -> 4
- board text added: "5V"
- board text added: "ANT"
- board text added: "F0"
- board text added: "F1"
- board text added: "FWD"
- board text added: "G"
- board text added: "KC1FSZ 2025-02"
- board text added: "REV"
- board text added: "RX"
- board text added: "TR"
- board text added: "TX"

Commit message: Sending QRP PA/LPF boards to JLC
Parts:
- added R10: 0, Resistor_SMD:R_0805_2012Metric_Pad1.20x1.40mm_HandSolder, F.Cu at (203.0, 78.2)
- added R9: 0, Resistor_SMD:R_0805_2012Metric_Pad1.20x1.40mm_HandSolder, F.Cu at (208.5, 78.2)
- moved C17 1.00 mm to (208.5, 73.5)
- moved C18 1.00 mm to (203.0, 73.5)
- moved D6 1.00 mm to (208.5, 71.0)
- moved D7 1.00 mm to (203.0, 71.0)
- moved R5 1.00 mm to (208.5, 68.5)
- moved R6 1.00 mm to (203.0, 68.5)
- moved R7 1.00 mm to (208.5, 76.0)
- moved R8 1.00 mm to (203.0, 76.0)
Connections:
- C17 pad 1: V_FWD -> Net-(D6-K)
- C18 pad 1: V_REV -> Net-(D7-K)
- D6 pad 1: V_FWD -> Net-(D6-K)
- D7 pad 1: V_REV -> Net-(D7-K)
- R7 pad 1: V_FWD -> Net-(D6-K)
- R8 pad 1: V_REV -> Net-(D7-K)
Routing:
- net Net-(D7-K): track 0.00 -> 7.52 mm
- net Net-(D6-K): track 0.00 -> 7.52 mm
- net V_REV: track 10.8 -> 3.42 mm
- net V_FWD: track 10.6 -> 3.25 mm
- net Net-(D7-A): track 23.5 -> 22.5 mm
- net Net-(D6-A): track 18.0 -> 17.0 mm
