File: hw/lpf1/lpf1.kicad_sch (KiCad schematic)
At the start: 39 parts, among them Q1 MMBT3904, Q2 MMBT3904, Q3 BS170F

Commit message: Layout in process
Parts:
- removed Q3: BS170F, Package_TO_SOT_SMD:SOT-23, symbol Transistor_FET:BS170F
- added C16, C9: 0.1uF, Capacitor_SMD:C_0805_2012Metric_Pad1.18x1.45mm_HandSolder, symbol Device:C_Small
- added D5: 1N4148W, Diode_SMD:D_SOD-123, symbol Diode:1N4148W
- added H1, H2, H3, H4: MountingHole, MountingHole:MountingHole_3.5mm, symbol Mechanical:MountingHole
- added J1, J2, J3: Conn_Coaxial, Connector_Coaxial:SMA_Amphenol_901-144_Vertical, symbol Connector:Conn_Coaxial
- added J4: Conn_01x05, Connector_PinHeader_2.54mm:PinHeader_1x05_P2.54mm_Vertical, symbol Connector_Generic:Conn_01x05
- added K1: G6E, Relay_THT:Relay_SPDT_Omron_G6E, symbol Relay:G6E
- added Q3: MMBT3904, Package_TO_SOT_SMD:SOT-23, symbol Transistor_BJT:MMBT3904
- C1, C10, C11, C12, C13, C14, C15, C2, C3, C4, C5, C6, C7, C8: footprint (none) -> Capacitor_SMD:C_0805_2012Metric_Pad1.18x1.45mm_HandSolder
- D1, D2, D3, D4: footprint (none) -> Diode_SMD:D_SOD-523
- L1, L10, L11, L12, L2, L3: footprint (none) -> bruce-footprints:FT37-43 Unifilar
- L13, L14, L4, L5, L6, L7, L8, L9: footprint (none) -> Inductor_SMD:L_0805_2012Metric_Pad1.15x1.40mm_HandSolder
- R1: value 560 -> 220; footprint (none) -> Resistor_SMD:R_0805_2012Metric_Pad1.20x1.40mm_HandSolder
- R2, R3: footprint (none) -> Resistor_SMD:R_0805_2012Metric_Pad1.20x1.40mm_HandSolder
- R4: value 10k -> 1k; footprint (none) -> Resistor_SMD:R_0805_2012Metric_Pad1.20x1.40mm_HandSolder
Connections:
- net GND: now also J1.2 (Ext), J2.2 (Ext), J3.2 (Ext), J4.5 (Pin_5), Q3.2 (E)
- net LPF_OUT: now also C16.2, J3.1 (In)
- net LPF_SEL0: now also J4.3 (Pin_3)
- net LPF_SEL1: now also J4.4 (Pin_4)
- net at C4.1, D2.2 (A), L6.1: no longer D3.2 (A), L8.1
- net at C1.1, D1.2 (A), L4.1: no longer D4.2 (A), L14.1
- net at R4.2: now also Q3.1 (B); no longer C4.2
- net +12V renamed +5V
- net +5V: now also D5.1 (K), J4.1 (Pin_1), K1.1; no longer R4.1
- new net: C9.1, D3.2 (A), L8.1
- new net: C16.1, D4.2 (A), L14.1
- new net: D5.2 (A), K1.6, Q3.3 (C)
- new net RF_A: C4.2, C9.2, K1.7
- new net RX_OUT: J2.1 (In), K1.10
- new net TX_IN: J1.1 (In), K1.12
- new net TX_SEL: J4.2 (Pin_2), R4.1
Other:
- note added: "Master T/R Relay (2A, 5V Coil)"
- note added: "Sets the bias current for PIN diodes. Two are connected at a time, so 5V / (10ma * 2) = 250 ohms"
- note removed: "Sets the bias current for PIN diodes. Two are connected at a time, so 12V / (10ma * 2) = 600 ohms"
- moved on the sheet: C1, C4

Commit message: Layout complete
Parts:
- removed C1, C10, C15, C16, C2, C3, C4, C9: 0.1uF, Capacitor_SMD:C_0805_2012Metric_Pad1.18x1.45mm_HandSolder, symbol Device:C_Small
- removed C11, C14: 180p, Capacitor_SMD:C_0805_2012Metric_Pad1.18x1.45mm_HandSolder, symbol Device:C_Small
- removed C12: 390p, Capacitor_SMD:C_0805_2012Metric_Pad1.18x1.45mm_HandSolder, symbol Device:C_Small
- removed C13: 390, Capacitor_SMD:C_0805_2012Metric_Pad1.18x1.45mm_HandSolder, symbol Device:C_Small
- removed C5, C6: 270p, Capacitor_SMD:C_0805_2012Metric_Pad1.18x1.45mm_HandSolder, symbol Device:C_Small
- removed C7, C8: 680p, Capacitor_SMD:C_0805_2012Metric_Pad1.18x1.45mm_HandSolder, symbol Device:C_Small
- removed D1, D2, D3, D4: D, Diode_SMD:D_SOD-523, symbol Device:D
- removed L1, L3: 1.38uH, bruce-footprints:FT37-43 Unifilar, symbol Device:L_Small
- removed L10, L12: 0.773u, bruce-footprints:FT37-43 Unifilar, symbol Device:L_Small
- removed L11: 0.904u, bruce-footprints:FT37-43 Unifilar, symbol Device:L_Small
- removed L13, L14, L4, L5, L6, L7, L8, L9: 47uH, Inductor_SMD:L_0805_2012Metric_Pad1.15x1.40mm_HandSolder, symbol Device:L_Small
- removed L2: 1.7uH, bruce-footprints:FT37-43 Unifilar, symbol Device:L_Small
- removed Q1, Q2: MMBT3904, Package_TO_SOT_SMD:SOT-23, symbol Transistor_BJT:MMBT3904
- removed R1: 220, Resistor_SMD:R_0805_2012Metric_Pad1.20x1.40mm_HandSolder, symbol Device:R_Small_US
- removed R2, R3: 1k, Resistor_SMD:R_0805_2012Metric_Pad1.20x1.40mm_HandSolder, symbol Device:R_Small_US
- added J5: Conn_01x04, Connector_PinHeader_2.54mm:PinHeader_1x04_P2.54mm_Vertical, symbol Connector_Generic:Conn_01x04
Connections:
- net GND: now also J5.2 (Pin_2), J5.4 (Pin_4)
- net LPF_OUT renamed ANT
- net RF_A renamed LPF_IN
- new net V_FWD: J5.1 (Pin_1)
- new net V_REV: J5.3 (Pin_3)
Other:
- added sheet LPF (lpf.kicad_sch)
- added sheet Stockton Bridge (sb.kicad_sch)
- note removed: "20m LPF"
- note removed: "40m LPF"
- note removed: "Sets the bias current for PIN diodes. Two are connected at a time, so 5V / (10ma * 2) = 250 ohms"

Commit message: Sending QRP PA/LPF boards to JLC
Other:
- company: (none) -> Bruce MacKinnon, KC1FSZ
- title: (none) -> Low Pass Filter Board 1
Changed lines of the file:
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@@
 	(generator "eeschema")
 	(generator_version "8.0")
-	(paper "A4")
+	(paper "USLetter")
+	(title_block
+		(title "Low Pass Filter Board 1")
+		(date "2025-02-21")
+		(rev "1")
+		(company "Bruce MacKinnon, KC1FSZ")
+		(comment 1 "Copyright (C) Bruce MacKinnon, 2025")
+		(comment 2 "NOT FOR COMMERCIAL USE")
+	)
 	(junction
 		(at 76.2 71.12)
